Commit message: modify python interface

File: src/robots_description/urdf/armlike_quadrotor_base.urdf.xacro (robot description, xacro)
@@ -27,5 +27,5 @@
       <child link="z_link"/>
       <axis xyz = "0 0 1"/>
-      <limit lower="0" upper="3" effort="5" velocity="5"/>
+      <limit lower="0.5" upper="10" effort="5" velocity="5"/>
     </joint>
     <link name="z_link"/>
